File: PCB/CommBadge/CommBadge.kicad_pcb (KiCad board)
At the start: 2 copper layers, 49.7 x 31.7 mm, 48 parts, among them J1 Reset, J2 Battery, J3 TC2030-USB-NL-DS, J5 USB-C-Socket-H, Q1 CJ2301, SW2 SW_Push, U2 MAX98357A, U3 TP4054, U4 ME6211C33M5G-N, U5 L, U6 ESP32-S3-MINI-1, U7 R

Commit message: Images
Parts:
- removed REF**: Shadow, RevK:Shadow
Other:
- copper layers 2 -> 4

Commit message: Re-render
Other:
- copper layers 4 -> 2
Changed lines of the file:
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@@
 		(0 "F.Cu" signal)
 		(2 "B.Cu" signal)
-		(9 "F.Adhes" user)
-		(11 "B.Adhes" user)
+		(9 "F.Adhes" user "F.Adhesive")
+		(11 "B.Adhes" user "B.Adhesive")
 		(13 "F.Paste" user)
 		(15 "B.Paste" user)
-		(5 "F.SilkS" user)
-		(7 "B.SilkS" user)
+		(5 "F.SilkS" user "F.Silkscreen")
+		(7 "B.SilkS" user "B.Silkscreen")
 		(1 "F.Mask" user)
 		(3 "B.Mask" user)
-		(17 "Dwgs.User" user)
-		(19 "Cmts.User" user)
-		(21 "Eco1.User" user)
-		(23 "Eco2.User" user)
+		(17 "Dwgs.User" user "User.Drawings")
+		(19 "Cmts.User" user "User.Comments")
+		(21 "Eco1.User" user "User.Eco1")
+		(23 "Eco2.User" user "User.Eco2")
 		(25 "Edge.Cuts" user)
 		(27 "Margin" user)
-		(31 "F.CrtYd" user)
-		(29 "B.CrtYd" user)
+		(31 "F.CrtYd" user "F.Courtyard")
+		(29 "B.CrtYd" user "B.Courtyard")
 		(35 "F.Fab" user)
 		(33 "B.Fab" user)
-		(39 "User.1" signal)
-		(41 "User.2" signal)
+		(39 "User.1" auxiliary)
+		(41 "User.2" auxiliary)
 	)
 	(setup
@@
 			(layer "F.Mask"
 				(type "Top Solder Mask")
-				(color "Purple")
+				(color "Blue")
 				(thickness 0.01)
 			)
