File: PCB/CommBadge/CommBadge.kicad_sch (KiCad schematic)
At the start: 47 parts, among them J1 Reset, J2 Battery, J3 TC2030-USB-NL-DS, J5 USB-C-Socket-H, Q1 CJ2301, SW2 SW_Push, U2 ESP32-S3-MINI-1, U2 MAX98357A, U3 TP4054, U4 ME6211C33M5G-N, U5 L, U7 R

Commit message: Re-render
Parts:
- renumbered C3 to C9, R1 to R2, U2 to U6
Changed lines of the file:
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@@
 (kicad_sch
-	(version 20231120)
+	(version 20241209)
 	(generator "eeschema")
-	(generator_version "8.0")
+	(generator_version "9.0")
 	(paper "A4")
 	(title_block
@@
 		(dnp no)
 		(fields_autoplaced yes)
-		(property "Reference" "#PWR0105"
+		(property "Reference" "#PWR022"
 			(at 80.01 118.745 0)
 			(effects
@@
 		(dnp no)
 		(fields_autoplaced yes)
-		(property "Reference" "U2"
+		(property "Reference" "U6"
 			(at 50.8 43.6332 0)
 			(effects
@@
 		(dnp no)
 		(fields_autoplaced yes)
-		(property "Reference" "#PWR03"
+		(property "Reference" "#PWR019"
 			(at 62.23 55.88 0)
 			(effects
@@
 		(dnp no)
 		(fields_autoplaced yes)
-		(property "Reference" "#PWR0106"
+		(property "Reference" "#PWR021"
 			(at 80.01 100.965 0)
 			(effects
@@
 		(dnp no)
 		(fields_autoplaced yes)
-		(property "Reference" "#PWR01"
+		(property "Reference" "#PWR020"
 			(at 72.39 60.96 0)
 			(effects
@@
 		(on_board yes)
 		(dnp no)
-		(property "Reference" "R1"
+		(property "Reference" "R2"
 			(at 81.915 100.965 90)
 			(effects
@@
 		(dnp no)
 		(fields_autoplaced yes)
-		(property "Reference" "C3"
+		(property "Reference" "C9"
 			(at 82.931 107.7503 0)
 			(effects
@@
 		)
 	)
+	(embedded_fonts no)
 )

Commit message: PCB Update
Parts:
- C1: footprint RevK:CP_EIA-3528-21_Kemet-B -> (none); JLCPCB Rotation Offset 180 -> (none); LCSC Part # C122649 -> (none)
- C10, C11, C12, C14, C15, C16, C17, C18, C2, C6, C9: footprint RevK:C_0402 -> (none)
- C13, C7, C8: footprint RevK:C_0402 -> (none); LCSC Part # C15525 -> (none)
- C3: footprint RevK:C_0603 -> (none)
- C4: footprint RevK:C_0805 -> (none); LCSC Part # C141660 -> (none)
- C5: footprint RevK:C_0603 -> (none); LCSC Part # C194427 -> (none)
- D1, D3: LCSC Part # C5137770 -> (none); MPN (none) -> C5137770
- D2: footprint RevK:D_SOD-123 -> (none); LCSC Part  C5204746 -> (none); MPN (none) -> C5204746
- D4, D5, D6, D7, D8, D9: footprint RevK:SMD1010 -> (none); LCSC Part # C5349953 -> (none); MPN (none) -> C5349953
- J1: footprint RevK:AA-Pad -> (none)
- J2: footprint RevK:1.25T-2PWT (Molex 532610271) -> (none); LCSC Part # C177225 -> (none)
- J5: LCSC Part # C709357 -> (none); MPN (none) -> C709357
- LS1: footprint RevK:KLJ-Speaker -> (none); LCSC Part # C18186315 -> (none)
- Q1: JLCPCB Rotation Offset 180 -> (none); LCSC Part # C5224170 -> (none)
- R1, R2, R3, R4, R5, R6, R8: footprint RevK:R_0402 -> (none)
- SW2: footprint RevK:TS-1092S-B3D2-G -> (none)
- U2: MPN (none) -> C2682619
- U3: JLCPCB Rotation Offset 180 -> (none); LCSC Part # C668215 -> (none); MPN (none) -> C668215
- U4: JLCPCB Rotation Offset -90 -> (none); LCSC Part # C82942 -> (none)
- U5, U7: LCSC Part # C5656610 -> (none); MPN (none) -> C5656610
- U6: LCSC Part # C3013941 -> (none); MPN (none) -> C3013941
