File: PCB/OSC/OCS.kicad_sch (KiCad schematic)
At the start: 44 parts, among them J1 Reset, J2 Wago, J3 TC2030-USB-NL-DS, J4 DC, J5 USB-C-Socket-H, J6 RELAY1, J7 RELAY2, SW1 SW_Push, SW2 SW_Reed, SW3 SW_Push, U1 ICS43434_MEMS_Mic, U2 ESP32-S3-MINI-1, U3 Relay, U4 78L05, U5 MD8942, U8 Relay, U9 VEML6040

Commit message: PCB Update
Parts:
- C1: footprint RevK:CP_EIA-3528-21_Kemet-B -> (none); JLCPCB Rotation Offset 180 -> (none); LCSC Part # C122649 -> (none)
- C10: renamed from C6; footprint RevK:C_0603_ -> (none); LCSC Part # C194427 -> (none)
- C11: renamed from C7; footprint RevK:C_0603_ -> (none); LCSC Part # C1691 -> (none)
- C12: renamed from C8; footprint RevK:C_0603_ -> (none)
- C15, C2: footprint RevK:C_0402 -> (none)
- C3: footprint RevK:C_0603 -> (none)
- C5: footprint RevK:C_0603 -> (none); LCSC Part # C194427 -> (none)
- C7, C8: footprint RevK:C_0402 -> (none); LCSC Part # C15525 -> (none)
- C9: renamed from C3; footprint RevK:C_0402 -> (none)
- D1: renamed from D4; footprint RevK:SMD1010 -> (none); LCSC Part # C5349953 -> (none); MPN (none) -> C5349953
- D2, D3, D4, D5: value ~ -> (none); LCSC Part # C5137770 -> (none); MPN (none) -> C5137770
- J1: footprint RevK:AA-Pad -> (none)
- J2: footprint RevK:WAGO-2060-453-998-404 -> (none); LCSC Part # C2765056 -> (none)
- J4, J6, J7: footprint RevK:WAGO-2060-452-998-404 -> (none); LCSC Part # C2765055 -> (none)
- J5: LCSC Part # C709357 -> (none); MPN (none) -> C709357
- L2: footprint RevK:L_4x4_ -> (none)
- R1, R10, R3, R5, R6, R7: footprint RevK:R_0402 -> (none)
- R14: renamed from R10; footprint RevK:R_0402_ -> (none)
- R15: renamed from R11; footprint RevK:R_0402_ -> (none)
- R2: renamed from R1; footprint RevK:R_0402 -> (none)
- R4: renamed from R9; footprint RevK:R_0402_ -> (none)
- SW1, SW3: footprint RevK:TS-1092S-B3D2-G -> (none)
- SW2: footprint RevK:Reed-59170 -> (none); LCSC Part # C315909 -> (none)
- U1: LCSC Part # C5656610 -> (none); MPN (none) -> C5656610
- U3, U8: JLCPCB Rotation Offset 180 -> (none); LCSC Part # C2691608 -> (none)
- U4: LCSC Part # C22392284 -> (none); MPN (none) -> C22392284
- U6: renamed from U2; LCSC Part # C3013941 -> (none); MPN (none) -> C3013941
- U7: renamed from U5; LCSC Part # C2684786 -> (none); MPN (none) -> C2684786
- U9: JLCPCB Rotation Offset 90 -> (none); LCSC Part # C78465 -> (none); MPN (none) -> C78465
