File: PCB/Recorder/Recorder.kicad_sch (KiCad schematic)
At the start: 47 parts, among them J1 Battery, J2 Reset, J3 TC2030-USB-NL-DS, J4 TF_PUSH, J5 USB-C-Socket-H, Q2 CJ2301, SW1 SW_Push, U1 R, U2 ESP32-S3-MINI-1, U2 L, U3 TP4054, U4 ME6211C33M5G-N

Commit message: Tidy
Parts:
- SW1: LCSC Part # (none) -> C520860
Changed lines of the file:
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@@
 			)
 		)
-		(property "Description" ""
+		(property "Description" "https://www.lcsc.com/datasheet/lcsc_datasheet_2409302331_Yuandi-TS-1092S-B3D2-G_C520860.pdf"
 			(at 270.51 65.405 0)
 			(effects
+				(font
+					(size 1.27 1.27)
+				)
+				(hide yes)
+			)
+		)
+		(property "LCSC Part #" "C520860"
+			(at 270.51 65.405 0)
+			(effects

Commit message: Re-order
Parts:
- renumbered C3 to C9, D4 to D1, R1 to R2, U2 to U6
Changed lines of the file:
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@@
 (kicad_sch
-	(version 20231120)
+	(version 20241209)
 	(generator "eeschema")
-	(generator_version "8.0")
+	(generator_version "9.0")
 	(paper "A4")
 	(title_block
@@
 		(dnp no)
 		(fields_autoplaced yes)
-		(property "Reference" "#PWR0105"
+		(property "Reference" "#PWR022"
 			(at 80.01 118.745 0)
 			(effects
@@
 		(dnp no)
 		(fields_autoplaced yes)
-		(property "Reference" "U2"
+		(property "Reference" "U6"
 			(at 50.8 43.6332 0)
 			(effects
@@
 		(dnp no)
 		(fields_autoplaced yes)
-		(property "Reference" "#PWR03"
+		(property "Reference" "#PWR019"
 			(at 62.23 55.88 0)
 			(effects
@@
 		(dnp no)
 		(fields_autoplaced yes)
-		(property "Reference" "#PWR0106"
+		(property "Reference" "#PWR021"
 			(at 80.01 100.965 0)
 			(effects
@@
 		(dnp no)
 		(fields_autoplaced yes)
-		(property "Reference" "#PWR01"
+		(property "Reference" "#PWR020"
 			(at 72.39 60.96 0)
 			(effects
@@
 		(on_board yes)
 		(dnp no)
-		(property "Reference" "D4"
+		(property "Reference" "D1"
 			(at 255.27 26.67 0)
 			(do_not_autoplace yes)
@@
 		(on_board yes)
 		(dnp no)
-		(property "Reference" "R1"
+		(property "Reference" "R2"
 			(at 81.915 100.965 90)
 			(effects
@@
 		(dnp no)
 		(fields_autoplaced yes)
-		(property "Reference" "#PWR019"
+		(property "Reference" "#PWR09"
 			(at 255.27 36.83 0)
 			(effects
@@
 		(dnp no)
 		(fields_autoplaced yes)
-		(property "Reference" "C3"
+		(property "Reference" "C9"
 			(at 82.931 107.7503 0)
 			(effects
@@
 		)
 	)
+	(embedded_fonts no)
 )

Commit message: Re-render
Parts:
- U1, U2: footprint RevK:ICS43434_MEMS_Mic_Open -> RevK:ICS43434_MEMS_Mic
- U4: footprint RevK:SOT-23-5 -> Package_TO_SOT_SMD:SOT-23-5; JLCPCB Rotation Offset -90 -> (none); Rotation Offset (none) -> 90
Changed lines of the file:
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@@
 			)
 		)
-		(property "Description" ""
+		(property "Description" "-0.33A Id, -60V Vds, P-Channel MOSFET, SOT-23"
 			(at 180.975 128.905 0)
 			(effects
@@
 			)
 		)
-		(property "Description" ""
+		(property "Description" "Resistor"
 			(at 114.3 66.675 0)
 			(effects
@@
 			)
 		)
-		(property "Description" ""
+		(property "Description" "Power symbol creates a global label with name \"GND\" , ground"
 			(at 204.47 136.525 0)
 			(effects
@@
 			)
 		)
-		(property "Description" ""
+		(property "Description" "Micro SD Card Socket"
 			(at 161.29 81.915 0)
 			(effects
@@
 			)
 		)
-		(property "Description" ""
+		(property "Description" "Resistor"
 			(at 121.92 66.675 0)
 			(effects
@@
 			)
 		)
-		(property "Description" ""
+		(property "Description" "Unpolarized capacitor"
 			(at 74.295 132.715 0)
 			(effects
@@
 			)
 		)
-		(property "Footprint" "RevK:ICS43434_MEMS_Mic_Open"
+		(property "Footprint" "RevK:ICS43434_MEMS_Mic"
 			(at 216.916 42.545 0)
 			(effects
@@
 			)
 		)
-		(property "Description" ""
+		(property "Description" "Special symbol for telling ERC where power comes from"
 			(at 190.5 126.365 0)
 			(effects
@@
 			)
 		)
-		(property "Footprint" "RevK:SOT-23-5"
+		(property "Footprint" "Package_TO_SOT_SMD:SOT-23-5"
 			(at 204.47 120.65 0)
 			(effects
@@
 			)
 		)
-		(property "Description" ""
+		(property "Description" "200mA Low Dropout Voltage Regulator, Fixed Output 3.3V, SOT-23-5"
 			(at 204.47 128.905 0)
 			(effects
@@
 			)
 		)
-		(property "JLCPCB Rotation Offset" "-90"
+		(property "Rotation Offset" "90"
 			(at 204.47 128.905 0)
 			(effects
@@
 			)
 		)
-		(property "Description" ""
+		(property "Description" "Resistor"
 			(at 133.35 66.675 0)
 			(effects
@@
 			)
 		)
-		(property "Description" ""
+		(property "Description" "Resistor"
 			(at 125.73 66.675 0)
 			(effects
@@
 			)
 		)
-		(property "Description" ""
+		(property "Description" "Schottky diode"
 			(at 189.865 133.985 0)
 			(effects
@@
 			)
 		)
-		(property "Description" ""
+		(property "Description" "Unpolarized capacitor"
 			(at 46.99 132.08 0)
 			(effects
@@
 			)
 		)
-		(property "Description" ""
+		(property "Description" "Battery charger"
 			(at 139.7 132.715 0)
 			(effects
@@
 			)
 		)
-		(property "Description" ""
+		(property "Description" "Unpolarized capacitor"
 			(at 271.145 45.72 0)
 			(effects
@@
 			)
 		)
-		(property "Description" ""
+		(property "Description" "Power symbol creates a global label with name \"GND\" , ground"
 			(at 180.975 141.605 0)
 			(effects
@@
 			)
 		)
-		(property "Description" ""
+		(property "Description" "Resistor"
 			(at 129.54 66.675 0)
 			(effects
@@
 			)
 		)
-		(property "Description" ""
+		(property "Description" "Resistor"
 			(at 137.16 66.675 0)
 			(effects
@@
 			)
 		)
-		(property "Datasheet" " ~"
+		(property "Datasheet" "~"
 			(at 132.08 34.925 0)
 			(effects
@@
 			)
 		)
-		(property "Description" ""
+		(property "Description" "Power symbol creates a global label with name \"GND\" , ground"
 			(at 181.61 97.155 0)
 			(effects
@@
 			)
 		)
-		(property "Datasheet" ""
+		(property "Datasheet" "~"
 			(at 148.59 165.1 0)
 			(effects
@@
 			)
 		)
-		(property "Description" ""
+		(property "Description" "Generic connector, single row, 01x02, script generated (kicad-library-utils/schlib/autogen/connector/)"
 			(at 148.59 165.1 0)
 			(effects
@@
 			)
 		)
-		(property "Description" ""
+		(property "Description" "Unpolarized capacitor"
 			(at 276.86 26.67 0)
 			(effects
@@
 			)
 		)
-		(property "Footprint" "RevK:ICS43434_MEMS_Mic_Open"
+		(property "Footprint" "RevK:ICS43434_MEMS_Mic"
 			(at 216.916 73.66 0)
 			(effects
@@
 			)
 		)
-		(property "Description" ""
+		(property "Description" "Resistor"
 			(at 118.11 66.675 0)
 			(effects
@@
 			)
 		)
-		(property "Description" ""
+		(property "Description" "Power symbol creates a global label with name \"GND\" , ground"
 			(at 275.59 65.405 0)
 			(effects
@@
 			)
 		)
-		(property "Description" ""
+		(property "Description" "Unpolarized capacitor"
 			(at 271.145 26.67 0)
 			(effects
@@
 			)
 		)
-		(property "Description" ""
+		(property "Description" "Power symbol creates a global label with name \"GND\" , ground"
 			(at 139.7 139.7 0)
 			(effects
@@
 			)
 		)
-		(property "Description" ""
+		(property "Description" "Power symbol creates a global label with name \"GND\" , ground"
 			(at 134.62 157.48 0)
 			(effects
@@
 			)
 		)
-		(property "Description" ""
+		(property "Description" "Unpolarized capacitor"
 			(at 239.395 92.075 0)
 			(effects
@@
 			)
 		)
-		(property "Description" "https://www.lcsc.com/datasheet/lcsc_datasheet_2409302331_Yuandi-TS-1092S-B3D2-G_C520860.pdf"
+		(property "Description" "Push button switch, generic, two pins"
 			(at 270.51 65.405 0)
 			(effects
@@
 			)
 		)
-		(property "Description" ""
+		(property "Description" "Unpolarized capacitor"
 			(at 215.265 133.985 0)
 			(effects
@@
 			)
 		)
-		(property "Description" ""
+		(property "Description" "Power symbol creates a global label with name \"GND\" , ground"
 			(at 130.175 142.24 0)
 			(effects
@@
 			)
 		)
-		(property "Description" ""
+		(property "Description" "Unpolarized capacitor"
 			(at 276.86 45.72 0)
 			(effects
@@
 			)
 		)
-		(property "Description" ""
+		(property "Description" "Unpolarized capacitor"
 			(at 239.395 60.96 0)
 			(effects
@@
 			)
 		)
-		(property "Description" ""
+		(property "Description" "Unpolarized capacitor"
 			(at 40.64 132.08 0)
 			(effects
@@
 			)
 		)
-		(property "Description" ""
+		(property "Description" "Resistor"
 			(at 130.175 138.43 0)
 			(effects
@@
 			)
 		)
-		(property "Description" ""
+		(property "Description" "Power symbol creates a global label with name \"GND\" , ground"
 			(at 215.265 137.795 0)
 			(effects
@@
 			)
 		)
-		(property "Description" ""
+		(property "Description" "Resistor"
 			(at 180.975 137.795 0)
 			(effects
@@
 			)
 		)
-		(property "Description" ""
+		(property "Description" "Unpolarized capacitor"
 			(at 91.44 133.35 0)
 			(effects
@@
 			)
 		)
-		(property "Description" ""
+		(property "Description" "Power symbol creates a global label with name \"+3.3V\""
 			(at 217.805 126.365 0)
 			(effects

Commit message: Tidy readme
Parts:
- U4: footprint Package_TO_SOT_SMD:SOT-23-5 -> RevK:SOT-23-5
Changed lines of the file:
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@@
 			)
 		)
-		(property "Footprint" "Package_TO_SOT_SMD:SOT-23-5"
+		(property "Footprint" "RevK:SOT-23-5"
 			(at 204.47 120.65 0)
 			(effects

Commit message: Cleanup for latest kicad
Parts:
- C1: JLCPCB Rotation Offset 180 -> (none); LCSC Part # C122649 -> (none); MPN (none) -> C122649
- D1, D4, D5, D6: MPN (none) -> C5349953
- J1: LCSC Part # C177225 -> (none); MPN (none) -> C177225
- J4: JLCPCB Position Offset 0,3.075 -> (none); MPN (none) -> C393941; Position Offset (none) -> 0,3.075
- J5: MPN (none) -> C709357
- U1, U2: MPN (none) -> C5656610
- U4: LCSC Part # C82942 -> (none); MPN (none) -> C82942
- U6: MPN (none) -> C3013941
Changed lines of the file:
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@@
 			)
 		)
-		(property "JLCPCB Position Offset" "0,3.075"
+		(property "Position Offset" "0,3.075"
+			(at 161.29 81.915 0)
+			(effects
+				(font
+					(size 1.27 1.27)
+				)
+				(hide yes)
+			)
+		)
+		(property "MPN" "C393941"
 			(at 161.29 81.915 0)
 			(effects
@@
 			)
 		)
+		(property "MPN" "C5656610"
+			(at 223.52 69.723 0)
+			(effects
+				(font
+					(size 1.27 1.27)
+				)
+				(hide yes)
+			)
+		)
 		(pin "6"
 		)
@@
 			)
 		)
-		(property "LCSC Part #" "C82942"
+		(property "MPN" "C82942"
 			(at 204.47 128.905 0)
 			(effects
@@
 			)
 		)
+		(property "MPN" "C5349953"
+			(at 264.16 15.24 0)
+			(effects
+				(font
+					(size 1 1)
+				)
+				(justify left top)
+				(hide yes)
+			)
+		)
 		(pin "1"
 		)
@@
 			)
 		)
+		(property "MPN" "C3013941"
+			(at 50.8 109.855 0)
+			(effects
+				(font
+					(size 1.27 1.27)
+				)
+				(hide yes)
+			)
+		)
 		(pin "1"
 		)
@@
 			)
 		)
+		(property "MPN" "C5349953"
+			(at 256.54 34.29 0)
+			(effects
+				(font
+					(size 1 1)
+				)
+				(justify left top)
+				(hide yes)
+			)
+		)
 		(pin "1"
 		)
@@
 			)
 		)
-		(property "LCSC Part #" "C177225"
+		(property "MPN" "C177225"
 			(at 148.59 165.1 0)
 			(effects
@@
 			)
 		)
+		(property "MPN" "C709357"
+			(at 247.65 130.175 0)
+			(effects
+				(font
+					(size 1.27 1.27)
+				)
+				(hide yes)
+			)
+		)
 		(pin "A1"
 		)
@@
 			)
 		)
-		(property "LCSC Part #" "C122649"
-			(at 52.705 132.08 0)
-			(effects
-				(font
-					(size 1.27 1.27)
-				)
-				(hide yes)
-			)
-		)
-		(property "JLCPCB Rotation Offset" "180"
+		(property "MPN" "C122649"
 			(at 52.705 132.08 0)
 			(effects
@@
 			)
 		)
+		(property "MPN" "C5656610"
+			(at 223.52 100.838 0)
+			(effects
+				(font
+					(size 1.27 1.27)
+				)
+				(hide yes)
+			)
+		)
 		(pin "6"
 		)
@@
 			)
 		)
+		(property "MPN" "C5349953"
+			(at 264.16 34.29 0)
+			(effects
+				(font
+					(size 1 1)
+				)
+				(justify left top)
+				(hide yes)
+			)
+		)
 		(pin "1"
 		)
@@
 			(at 256.54 15.24 0)
 			(effects
+				(font
+					(size 1 1)
+				)
+				(justify left top)
+				(hide yes)
+			)
+		)
+		(property "MPN" "C5349953"
+			(at 256.54 15.24 0)
+			(effects

Commit message: Fucking KiCAD changes
Parts:
- D2: MPN (none) -> C5137770
- D3: LCSC Part  C5204746 -> (none); MPN (none) -> C5204746
- J4: LCSC Part # C393941 -> (none); Position Offset 0,3.075 -> 0,0.15
- J5: value USB-C-Socket-H -> USB-C-Socket-V; Position Offset (none) -> 0,0.7
- U1, U2: footprint RevK:ICS43434_MEMS_Mic -> RevK:ICS43434_MEMS_Mic_Open
- U3: MPN (none) -> C668215; Rotation Offset (none) -> 180
Changed lines of the file:
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@@
 			)
 		)
-		(property "LCSC Part #" "C393941"
-			(at 161.29 81.915 0)
-			(effects
-				(font
-					(size 1.27 1.27)
-				)
-				(hide yes)
-			)
-		)
-		(property "Position Offset" "0,3.075"
+		(property "MPN" "C393941"
 			(at 161.29 81.915 0)
 			(effects
@@
 			)
 		)
-		(property "MPN" "C393941"
+		(property "Position Offset" "0,0.15"
 			(at 161.29 81.915 0)
 			(effects
@@
 			)
 		)
-		(property "Footprint" "RevK:ICS43434_MEMS_Mic"
+		(property "Footprint" "RevK:ICS43434_MEMS_Mic_Open"
 			(at 216.916 42.545 0)
 			(effects
@@
 			)
 		)
-		(property "LCSC Part " "C5204746"
+		(property "MPN" "C5204746"
 			(at 189.865 133.985 0)
 			(effects
@@
 			)
 		)
+		(property "MPN" "C668215"
+			(at 133.35 127 0)
+			(effects
+				(font
+					(size 1.27 1.27)
+				)
+				(hide yes)
+			)
+		)
+		(property "Rotation Offset" "180"
+			(at 130.81 125.095 0)
+			(effects
+				(font
+					(size 1.27 1.27)
+				)
+				(hide yes)
+			)
+		)
 		(pin "1"
 		)
@@
 			)
 		)
-		(property "Value" "USB-C-Socket-H"
+		(property "Value" "USB-C-Socket-V"
 			(at 247.65 110.6749 0)
 			(effects
@@
 			)
 		)
+		(property "Position Offset" "0,0.7"
+			(at 247.65 130.175 0)
+			(effects
+				(font
+					(size 1.27 1.27)
+				)
+				(hide yes)
+			)
+		)
 		(pin "A1"
 		)
@@
 			)
 		)
-		(property "Footprint" "RevK:ICS43434_MEMS_Mic"
+		(property "Footprint" "RevK:ICS43434_MEMS_Mic_Open"
 			(at 216.916 73.66 0)
 			(effects
@@
 			(at 142.24 161.29 0)
 			(effects
+				(font
+					(size 1.27 1.27)
+				)
+				(hide yes)
+			)
+		)
+		(property "MPN" "C5137770"
+			(at 142.24 161.29 0)
+			(effects

Commit message: PCB Update
Parts:
- C11, C7: LCSC Part # C15525 -> (none); MPN (none) -> C15525
- C16: LCSC Part # C141660 -> (none); MPN (none) -> C141660
- D1, D4, D5, D6: LCSC Part # C5349953 -> (none)
- D2: LCSC Part # C5137770 -> (none)
- J4: Position Offset 0,0.15 -> (none)
- J5: value USB-C-Socket-V -> USB-C-Socket-H; LCSC Part # C709357 -> (none); Position Offset 0,0.7 -> (none)
- Q2: JLCPCB Rotation Offset 180 -> (none); LCSC Part # C8547 -> (none); MPN (none) -> C8547
- SW1: LCSC Part # C520860 -> (none); MPN (none) -> C520860
- U1, U2: LCSC Part # C5656610 -> (none)
- U3: JLCPCB Rotation Offset 180 -> (none); LCSC Part # C668215 -> (none); Rotation Offset 180 -> (none)
- U4: MPN C82942 -> (none); Rotation Offset 90 -> (none)
- U6: LCSC Part # C3013941 -> (none)
Changed lines of the file:
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@@
 			)
 		)
-		(property "LCSC Part #" "C8547"
-			(at 180.975 128.905 90)
-			(effects
-				(font
-					(size 1.27 1.27)
-				)
-				(hide yes)
-			)
-		)
-		(property "JLCPCB Rotation Offset" "180"
+		(property "MPN" "C8547"
 			(at 180.975 128.905 90)
 			(effects
@@
 			)
 		)
-		(property "Position Offset" "0,0.15"
-			(at 161.29 81.915 0)
-			(effects
-				(font
-					(size 1.27 1.27)
-				)
-				(hide yes)
-			)
-		)
 		(pin "1"
 		)
@@
 			)
 		)
-		(property "LCSC Part #" "C15525"
+		(property "MPN" "C15525"
 			(at 74.295 132.715 0)
 			(effects
@@
 			)
 		)
-		(property "LCSC Part #" "C5656610"
-			(at 223.52 69.723 0)
-			(effects
-				(font
-					(size 1.27 1.27)
-				)
-				(hide yes)
-			)
-		)
 		(property "MPN" "C5656610"
 			(at 223.52 69.723 0)
@@
 			)
 		)
-		(property "MPN" "C82942"
-			(at 204.47 128.905 0)
-			(effects
-				(font
-					(size 1.27 1.27)
-				)
-				(hide yes)
-			)
-		)
-		(property "Rotation Offset" "90"
-			(at 204.47 128.905 0)
-			(effects
-				(font
-					(size 1.27 1.27)
-				)
-				(hide yes)
-			)
-		)
 		(pin "1"
 		)
@@
 			)
 		)
-		(property "LCSC Part #" "C5349953"
+		(property "MPN" "C5349953"
 			(at 264.16 15.24 0)
 			(effects
@@
 			)
 		)
-		(property "Description" ""
+		(property "Description" "ESP32S3"
 			(at 50.8 77.47 0)
 			(effects
@@
 			)
 		)
-		(property "LCSC Part #" "C3013941"
-			(at 50.8 109.855 0)
-			(effects
-				(font
-					(size 1.27 1.27)
-				)
-				(hide yes)
-			)
-		)
 		(property "MPN" "C3013941"
 			(at 50.8 109.855 0)
@@
 			)
 		)
-		(property "Datasheet" "https://www.lcsc.com/datasheet/lcsc_datasheet_2409241408_UMW-Youtai-Semiconductor-Co---Ltd--TP4054_C668215.pdf"
+		(property "Datasheet" ""
 			(at 139.7 132.715 0)
 			(effects
@@
 			)
 		)
-		(property "LCSC Part #" "C668215"
-			(at 133.35 127 0)
-			(effects
-				(font
-					(size 1.27 1.27)
-				)
-				(hide yes)
-			)
-		)
-		(property "JLCPCB Rotation Offset" "180"
-			(at 130.81 125.095 0)
-			(effects
-				(font
-					(size 1.27 1.27)
-				)
-				(hide yes)
-			)
-		)
 		(property "MPN" "C668215"
 			(at 133.35 127 0)
@@
 			)
 		)
-		(property "Rotation Offset" "180"
-			(at 130.81 125.095 0)
-			(effects
-				(font
-					(size 1.27 1.27)
-				)
-				(hide yes)
-			)
-		)
 		(pin "1"
 		)
@@
 			)
 		)
-		(property "LCSC Part #" "C5349953"
+		(property "MPN" "C5349953"
 			(at 256.54 34.29 0)
 			(effects
@@
 			)
 		)
-		(property "Value" "USB-C-Socket-V"
+		(property "Value" "USB-C-Socket-H"
 			(at 247.65 110.6749 0)
 			(effects
@@
 			)
 		)
-		(property "LCSC Part #" "C709357"
-			(at 247.65 130.175 0)
-			(effects
-				(font
-					(size 1.27 1.27)
-				)
-				(hide yes)
-			)
-		)
 		(property "MPN" "C709357"
 			(at 247.65 130.175 0)
@@
 			)
 		)
-		(property "Position Offset" "0,0.7"
-			(at 247.65 130.175 0)
-			(effects
-				(font
-					(size 1.27 1.27)
-				)
-				(hide yes)
-			)
-		)
 		(pin "A1"
 		)
@@
 			)
 		)
-		(property "LCSC Part #" "C5656610"
-			(at 223.52 100.838 0)
-			(effects
-				(font
-					(size 1.27 1.27)
-				)
-				(hide yes)
-			)
-		)
 		(property "MPN" "C5656610"
 			(at 223.52 100.838 0)
@@
 			)
 		)
-		(property "LCSC Part #" "C5349953"
+		(property "MPN" "C5349953"
 			(at 264.16 34.29 0)
 			(effects
@@
 			)
 		)
-		(property "LCSC Part #" "C5349953"
+		(property "MPN" "C5349953"
 			(at 256.54 15.24 0)
 			(effects
@@
 			)
 		)
-		(property "LCSC Part #" "C520860"
+		(property "MPN" "C520860"
 			(at 270.51 65.405 0)
 			(effects
@@
 			)
 		)
-		(property "LCSC Part #" "C141660"
+		(property "MPN" "C141660"
 			(at 215.265 133.985 0)
 			(effects
@@
 			)
 		)
-		(property "LCSC Part #" "C15525"
+		(property "MPN" "C15525"
 			(at 91.44 133.35 0)
 			(effects
@@
 			)
 		)
-		(property "LCSC Part #" "C5137770"
+		(property "MPN" "C5137770"
 			(at 142.24 161.29 0)
 			(effects

Commit message: Tidy
Connections:
- net D-: now also J3.2 (NC), J3.6 (NC)
- net GND: no longer J3.6 (GND)
- net VBUS: no longer J3.2 (VBUS)
