File: PCB/Recorder/Recorder.kicad_pcb (KiCad board)
At the start: 2 copper layers, 70 x 70 mm, 58 parts, among them J1 Reset, J3 TC2030-USB-NL-DS, J4 TF_PUSH, J5 USB-C-Socket-H, J6 Battery, Q1 CJ2301, SW1 SW_Push_DPDT, U1 ESP32-S3-MINI-1-N4R2, U2 TPS22916CNYFPR, U3 TP4054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

Commit message: Library update
Other:
- board text added: "3.7V LiPo"

Commit message: Case render fix
Parts:
- moved J6 1.50 mm to (120.2, 105.5)
Routing:
- net VBATCHG: track 31.1 -> 30.0 mm
- net Net-(J1-Pin_2): track 24.4 -> 25.0 mm
Other:
- board text added: "3.7V"
- board text removed: "3.7V LiPo"

Commit message: Revised for order
Routing:
- net D-: track 55.8 -> 55.2 mm
- net D+: track 54.7 -> 54.1 mm
- net GND: vias 39 -> 40

Commit message: Library update
Parts:
- moved BT1 1.50 mm to (106.0, 99.5)

Commit message: Loop
Routing:
- net GND: vias 40 -> 45
