File: PCB/Intercom/Intercom.kicad_sch (KiCad schematic)
At the start: 33 parts, among them J1 Reset, J2 Battery, J3 TC2030-USB-NL-DS, J5 USB-C-Socket-H, Q1 CJ2301, SW2 SW_Push, U2 ESP32-S3-MINI-1, U2 MAX98357A, U3 TP4054, U4 ME6211C33M5G-N, U5 L, U7 R

Commit message: PCB Update
Parts:
- C1: footprint RevK:CP_EIA-3528-21_Kemet-B -> (none); JLCPCB Rotation Offset 180 -> (none); LCSC Part # C122649 -> (none)
- C10, C14, C2, C6: footprint RevK:C_0402 -> (none)
- C13, C7, C8: footprint RevK:C_0402 -> (none); LCSC Part # C15525 -> (none)
- C3: footprint RevK:C_0603 -> (none)
- C4: footprint RevK:C_0805 -> (none); LCSC Part # C141660 -> (none)
- C5: footprint RevK:C_0603 -> (none); LCSC Part # C194427 -> (none)
- C9: renamed from C3; footprint RevK:C_0402 -> (none)
- D1, D3: LCSC Part # C5137770 -> (none); MPN (none) -> C5137770
- D2: footprint RevK:D_SOD-123 -> (none); LCSC Part  C5204746 -> (none); MPN (none) -> C5204746
- J1: footprint RevK:AA-Pad -> (none)
- J2: footprint RevK:1.25T-2PWT (Molex 532610271) -> (none); LCSC Part # C177225 -> (none)
- J5: LCSC Part # C709357 -> (none); MPN (none) -> C709357
- Q1: JLCPCB Rotation Offset 180 -> (none); LCSC Part # C5224170 -> (none)
- R1, R3, R5, R6, R8: footprint RevK:R_0402 -> (none)
- R2: renamed from R1; footprint RevK:R_0402 -> (none)
- SW2: footprint RevK:TS-1092S-B3D2-G -> (none)
- U2: MPN (none) -> C2682619
- U3: JLCPCB Rotation Offset 180 -> (none); LCSC Part # C668215 -> (none); MPN (none) -> C668215
- U4: JLCPCB Rotation Offset -90 -> (none); LCSC Part # C82942 -> (none)
- U5, U7: LCSC Part # C5656610 -> (none); MPN (none) -> C5656610
- U6: renamed from U2; LCSC Part # C3013941 -> (none); MPN (none) -> C3013941
Changed lines of the file:
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@@
 (kicad_sch
-	(version 20231120)
+	(version 20241209)
 	(generator "eeschema")
-	(generator_version "8.0")
+	(generator_version "9.0")
 	(paper "A4")
 	(title_block
@@
 			)
 		)
-		(property "Footprint" "RevK:R_0402"
+		(property "Footprint" ""
 			(at 231.14 37.338 90)
 			(effects
@@
 			)
 		)
-		(property "Footprint" "RevK:R_0402"
+		(property "Footprint" ""
 			(at 231.14 36.322 90)
 			(effects
@@
 		(dnp no)
 		(fields_autoplaced yes)
-		(property "Reference" "#PWR0105"
+		(property "Reference" "#PWR022"
 			(at 80.01 118.745 0)
 			(effects
@@
 			)
 		)
-		(property "Footprint" "RevK:C_0402"
+		(property "Footprint" ""
 			(at 79.7052 144.78 0)
 			(effects
@@
 			)
 		)
-		(property "LCSC Part #" "C15525"
-			(at 78.74 140.97 0)
-			(effects
-				(font
-					(size 1.27 1.27)
-				)
-				(hide yes)
-			)
-		)
 		(pin "1"
 		)
@@
 			)
 		)
-		(property "LCSC Part #" "C5224170"
-			(at 168.275 112.395 90)
-			(effects
-				(font
-					(size 1.27 1.27)
-				)
-				(hide yes)
-			)
-		)
-		(property "JLCPCB Rotation Offset" "180"
-			(at 168.275 112.395 90)
-			(effects
-				(font
-					(size 1.27 1.27)
-				)
-				(hide yes)
-			)
-		)
 		(pin "1"
 		)
@@
 			)
 		)
-		(property "Footprint" "RevK:C_0402"
+		(property "Footprint" ""
 			(at 259.3848 104.775 0)
 			(effects
@@
 			)
 		)
-		(property "Footprint" "RevK:1.25T-2PWT (Molex 532610271)"
+		(property "Footprint" ""
 			(at 135.89 148.59 0)
 			(effects
@@
 			)
 		)
-		(property "LCSC Part #" "C177225"
-			(at 135.89 148.59 0)
-			(effects
-				(font
-					(size 1.27 1.27)
-				)
-				(hide yes)
-			)
-		)
 		(pin "2"
 		)
@@
 			)
 		)
-		(property "LCSC Part #" "C5656610"
+		(property "MPN" "C5656610"
 			(at 242.57 117.348 0)
 			(effects
@@
 			)
 		)
-		(property "Footprint" "RevK:C_0603"
+		(property "Footprint" ""
 			(at 39.7002 144.78 0)
 			(effects
@@
 		(dnp no)
 		(fields_autoplaced yes)
-		(property "Reference" "U2"
+		(property "Reference" "U6"
 			(at 50.8 43.6332 0)
 			(effects
@@
 			)
 		)
-		(property "LCSC Part #" "C3013941"
+		(property "MPN" "C3013941"
 			(at 50.8 109.855 0)
 			(effects
@@
 			)
 		)
-		(property "Footprint" "RevK:C_0402"
+		(property "Footprint" ""
 			(at 168.6052 68.58 0)
 			(effects
@@
 		(dnp no)
 		(fields_autoplaced yes)
-		(property "Reference" "#PWR03"
+		(property "Reference" "#PWR019"
 			(at 62.23 55.88 0)
 			(effects
@@
 		(dnp no)
 		(fields_autoplaced yes)
-		(property "Reference" "#PWR0106"
+		(property "Reference" "#PWR021"
 			(at 80.01 100.965 0)
 			(effects
@@
 			)
 		)
-		(property "LCSC Part #" "C82942"
-			(at 191.77 112.395 0)
-			(effects
-				(font
-					(size 1.27 1.27)
-				)
-				(hide yes)
-			)
-		)
-		(property "JLCPCB Rotation Offset" "-90"
-			(at 191.77 112.395 0)
-			(effects
-				(font
-					(size 1.27 1.27)
-				)
-				(hide yes)
-			)
-		)
 		(pin "1"
 		)
@@
 			)
 		)
-		(property "Footprint" "RevK:C_0805"
+		(property "Footprint" ""
 			(at 203.5302 121.285 0)
 			(effects
@@
 			)
 		)
-		(property "LCSC Part #" "C141660"
-			(at 202.565 117.475 0)
-			(effects
-				(font
-					(size 1.27 1.27)
-				)
-				(hide yes)
-			)
-		)
 		(pin "1"
 		)
@@
 			)
 		)
-		(property "Footprint" "RevK:AA-Pad"
+		(property "Footprint" ""
 			(at 20.32 104.14 0)
 			(effects
@@
 			)
 		)
-		(property "Footprint" "RevK:C_0603"
+		(property "Footprint" ""
 			(at 63.1952 144.145 0)
 			(effects
@@
 			)
 		)
-		(property "LCSC Part #" "C194427"
-			(at 62.23 140.335 0)
-			(effects
-				(font
-					(size 1.27 1.27)
-				)
-				(hide yes)
-			)
-		)
 		(pin "1"
 		)
@@
 			)
 		)
-		(property "Footprint" "RevK:C_0402"
+		(property "Footprint" ""
 			(at 259.3848 135.89 0)
 			(effects
@@
 			)
 		)
-		(property "Footprint" "RevK:R_0402"
+		(property "Footprint" ""
 			(at 119.253 121.92 90)
 			(effects
@@
 			)
 		)
-		(property "Footprint" "RevK:TS-1092S-B3D2-G"
+		(property "Footprint" ""
 			(at 173.99 25.4 0)
 			(effects
@@
 			)
 		)
-		(property "Footprint" "RevK:R_0402"
+		(property "Footprint" ""
 			(at 145.542 69.215 90)
 			(effects
@@
 		(dnp no)
 		(fields_autoplaced yes)
-		(property "Reference" "#PWR01"
+		(property "Reference" "#PWR020"
 			(at 72.39 60.96 0)
 			(effects
@@
 			)
 		)
-		(property "LCSC Part #" "C709357"
+		(property "MPN" "C709357"
 			(at 209.55 45.72 0)
 			(effects
@@
 			)
 		)
-		(property "Footprint" "RevK:CP_EIA-3528-21_Kemet-B"
+		(property "Footprint" ""
 			(at 45.4152 144.78 0)
 			(effects
@@
 			)
 		)
-		(property "LCSC Part #" "C122649"
-			(at 44.45 140.97 0)
-			(effects
-				(font
-					(size 1.27 1.27)
-				)
-				(hide yes)
-			)
-		)
-		(property "JLCPCB Rotation Offset" "180"
-			(at 44.45 140.97 0)
-			(effects
-				(font
-					(size 1.27 1.27)
-				)
-				(hide yes)
-			)
-		)
 		(pin "1"
 		)
@@
 			)
 		)
-		(property "LCSC Part #" ""
+		(property "MPN" "C2682619"
 			(at 123.825 64.135 0)
 			(effects
@@
 					(size 1.27 1.27)
 				)
+				(hide yes)
 			)
 		)
@@
 			)
 		)
-		(property "Footprint" "RevK:C_0402"
+		(property "Footprint" ""
 			(at 91.7702 144.78 0)
 			(effects
@@
 			)
 		)
-		(property "LCSC Part #" "C15525"
-			(at 90.805 140.97 0)
-			(effects
-				(font
-					(size 1.27 1.27)
-				)
-				(hide yes)
-			)
-		)
 		(pin "1"
 		)
@@
 		(on_board yes)
 		(dnp no)
-		(property "Reference" "R1"
+		(property "Reference" "R2"
 			(at 81.915 100.965 90)
 			(effects
@@
 			)
 		)
-		(property "Footprint" "RevK:R_0402"
+		(property "Footprint" ""
 			(at 78.232 100.965 90)
 			(effects
@@
 			)
 		)
-		(property "Footprint" "RevK:D_SOD-123"
+		(property "Footprint" ""
 			(at 177.165 117.475 0)
 			(effects
@@
 			)
 		)
-		(property "LCSC Part " "C5204746"
+		(property "MPN" "C5204746"
 			(at 177.165 117.475 0)
 			(effects
@@
 					(size 1.27 1.27)
 				)
-				(hide yes)
 			)
 		)
@@
 			)
 		)
-		(property "Footprint" "RevK:C_0402"
+		(property "Footprint" ""
 			(at 33.3502 144.78 0)
 			(effects
@@
 			)
 		)
-		(property "LCSC Part #" "C5656610"
+		(property "MPN" "C5656610"
 			(at 242.57 148.463 0)
 			(effects
@@
 			)
 		)
-		(property "LCSC Part #" "C5137770"
+		(property "MPN" "C5137770"
 			(at 129.54 144.78 0)
 			(effects
@@
 		(dnp no)
 		(fields_autoplaced yes)
-		(property "Reference" "C3"
+		(property "Reference" "C9"
 			(at 82.931 107.7503 0)
 			(effects
@@
 			)
 		)
-		(property "Footprint" "RevK:C_0402"
+		(property "Footprint" ""
 			(at 80.9752 112.395 0)
 			(effects
@@
 			)
 		)
-		(property "Datasheet" "https://www.lcsc.com/datasheet/lcsc_datasheet_2409241408_UMW-Youtai-Semiconductor-Co---Ltd--TP4054_C668215.pdf"
+		(property "Datasheet" ""
 			(at 127 116.205 0)
 			(effects
@@
 			)
 		)
-		(property "LCSC Part #" "C668215"
+		(property "MPN" "C668215"
 			(at 120.65 110.49 0)
 			(effects
@@
 			)
 		)
-		(property "JLCPCB Rotation Offset" "180"
-			(at 118.11 108.585 0)
-			(effects
-				(font
-					(size 1.27 1.27)
-				)
-				(hide yes)
-			)
-		)
 		(pin "1"
 		)
@@
 			)
 		)
-		(property "LCSC Part #" "C5137770"
+		(property "MPN" "C5137770"
 			(at 173.99 37.465 0)
 			(effects
@@
 			)
 		)
-		(property "Footprint" "RevK:R_0402"
+		(property "Footprint" ""
 			(at 166.497 121.285 90)
 			(effects
@@
 			)
 		)
-		(property "Footprint" "RevK:C_0402"
+		(property "Footprint" ""
 			(at 156.5402 68.58 0)
 			(effects
@@
 			)
 		)
-		(property "LCSC Part #" "C15525"
-			(at 155.575 64.77 0)
-			(effects
-				(font
-					(size 1.27 1.27)
-				)
-				(hide yes)
-			)
-		)
 		(pin "1"
 		)
@@
 		)
 	)
+	(embedded_fonts no)
 )

Commit message: Started new Intercom
Parts:
- removed C1: 220uF Tant, symbol Device:C_Polarized
- removed C2: 100nF, symbol Device:C
- removed C3: 22uF, symbol Device:C
- removed C4: 100uF, symbol Device:C
- removed D1, D3: ~, RevK:DFN1006-2L, symbol RevK:ES05D1MC10
- removed D2: MBR0530, symbol Device:D_Schottky
- removed J2: Battery, symbol Connector_Generic:Conn_01x02
- removed Q1: CJ2301, RevK:SOT-23, symbol Transistor_FET:BSS83P
- removed R1, R3: 10K, symbol Device:R
- removed R8: 634K, symbol Device:R
- removed SW2: SW_Push, symbol Switch:SW_Push
- removed U3: TP4054, RevK:SOT-23-5, symbol RevK:TP4054
- removed U4: ME6211C33M5G-N, RevK:SOT-23-5, symbol Regulator_Linear:TLV70033_SOT23-5
- removed U5: L, RevK:ICS43434_MEMS_Mic_Open, symbol RevK:ICS43434_MEMS_Mic
- removed U7: R, RevK:ICS43434_MEMS_Mic_Open, symbol RevK:ICS43434_MEMS_Mic
- added C1: 10uF 35V, RevK:C_0603_, symbol RevK:Hidden
- added C11, C15, C9: 100nF, RevK:C_0402, symbol Device:C
- added C16: 22uF, RevK:C_0603, symbol Device:C
- added C2: 10uF 6.3V, RevK:C_0603_, symbol RevK:Hidden
- added C3: 100nF, RevK:C_0603_, symbol RevK:Hidden
- added D1, D2, D3, D4, D5, D6: XL-1010RGBC-WS2812B, RevK:SMD1010, symbol RevK:WS2812B-1mm
- added J2: JST-PH-SM4-TB, RevK:JST_PH_S2B-PH-SM4-TB_1x02-1MP_P2.00mm_Horizontal, symbol Connector_Generic:Conn_01x04
- added L1: 10uH, RevK:L_4x4_, symbol RevK:Hidden
- added PCB1: 70x70, RevK:PCB7070, symbol RevK:PCB
- added R1: 124k, RevK:R_0402_, symbol RevK:Hidden
- added R2: 39k2, RevK:R_0402_, symbol RevK:Hidden
- added R3: 1M, RevK:R_0402_, symbol RevK:Hidden
- added R4: 634K, symbol Device:R
- added SW1: SW_Push, RevK:TS-1092S-B3D2-G, symbol Switch:SW_Push
- added U1: MD8942, RevK:SOT-23-6-MD8942, symbol RevK:MD89420-RegBlock
- added U4: R, RevK:ICS43434_MEMS_Mic, symbol RevK:ICS43434_MEMS_Mic
- added V2, V3: ~, RevK:VCUT70N, symbol RevK:VCUT
- C10, C14, C6: footprint (none) -> RevK:C_0402
- C12: renamed from C13; footprint (none) -> RevK:C_0402; MPN (none) -> C15525
- C4: renamed from C9; footprint (none) -> RevK:C_0402
- C5: value 10uF 35V -> 100nF; footprint (none) -> RevK:C_0402
- C7, C8: value 10uF -> 100nF; footprint (none) -> RevK:C_0402
- J1: footprint (none) -> RevK:AA-Pad
- R6: renamed from R2; footprint (none) -> RevK:R_0402
- R7: renamed from R5; footprint (none) -> RevK:R_0402
- R8: renamed from R6; footprint (none) -> RevK:R_0402
- renumbered J3 to J4, U6 to U2, U2 to U6
Connections:
- net SKPPWR is gone; now on net MICSD: U2.40 (GPIO44)
- net +3V3: now also C15.1, C16.1, U1.8 (VOUT), U4.2 (LR), U4.5 (VDD); no longer C12.1, C14.1, C6.2, C7.1, C8.1, U6.A2 (VDD)
- net D-: now also J4.2 (NC), J4.6 (NC)
- net GND: now also C5.1, C7.1, C8.1, U6.B2 (GAIN_SLOT), C11.1, C15.2, C16.2, C9.1, D1.3 (-), D2.3 (-), D3.3 (-), D4.3 (-), D5.3 (-), D6.3 (-), J2.3 (Pin_3), J2.4 (Pin_4), SW1.1, U1.2 (GND), U1.7 (GND), U4.3 (GND); no longer C5.2, C7.2, C8.2, J4.6 (GND)
- net MICSCK: now also U2.39 (GPIO43), U4.4 (SCK); no longer U2.38 (GPIO42)
- net MICSD: now also U4.6 (SD); no longer U2.37 (GPIO41)
- net MICWS: now also U2.44 (GPIO46), U4.1 (WS); no longer U2.36 (GPIO40)
- net BTN: now reaches U2.10 (GPIO6)
- net BTN: now also SW1.2
- net at U6.A1 (~{SD_MODE}): now also R4.1
- net at U6.A3 (OUTP): now also J2.2 (Pin_2)
- net at U6.B3 (OUTN): now also J2.1 (Pin_1)
- net CHARGING renamed LED
- net LED: now also D3.4 (I)
- net DC renamed +5V
- net +5V: now also C12.1, C14.1, C5.2, C6.2, C7.2, C8.2, U6.A2 (VDD), C11.2, C9.2, D1.2 (+), D2.2 (+), D3.2 (+), D4.2 (+), D5.2 (+), D6.2 (+), U1.5 (VIN); no longer C5.1, J4.2 (VBUS)
- net PUSH: no longer names the net of U2.15 (GPIO11)
- net RGB renamed SPKPWR
- net SPKPWR: now also R4.2
- net SKPSCK renamed SPKBSCK
- net SKPSD renamed SPKDATA
- net SKPWS renamed SPKLRC
- new net: D5.1 (O), D6.4 (I)
- new net: D4.1 (O), D5.4 (I)
- new net: D2.1 (O), D4.4 (I)
- new net: D1.1 (O), D2.4 (I)
- new net: D1.4 (I), D3.1 (O)
- no-connect marks 26 -> 28
Other:
- title: Intercom -> IronMan Chest
- moved on the sheet: C12, C14, J5, R7, R8, U6

Commit message: New PCB
Parts:
- removed SW1: SW_Push, RevK:TS-1092S-B3D2-G, symbol Switch:SW_Push
- added C13, C17, C18, C19, C21, C22, C23, C24, C25, C26, C27, C28, C29, C30: 100nF, RevK:C_0402, symbol Device:C
- added C20: 220uF Tant, RevK:CP_EIA-3528-21_Kemet-B, symbol Device:C_Polarized
- added C31: C_Polarized, RevK:CP_EIA-7343-31_Kemet-D, symbol Device:C_Polarized
- added D10, D11, D12, D13, D14, D15, D16, D17, D18, D19, D20, D7, D8, D9: XL-1010RGBC-WS2812B, RevK:SMD1010, symbol RevK:WS2812B-1mm
- added P1, P2: Square, RevK:PAD-2mm, symbol RevK:Square
- added SW1: SW_SPST, RevK:SPEH130103, symbol Switch:SW_SPST
- R4: footprint (none) -> RevK:R_0402
- U4: value R -> ICS43434; footprint RevK:ICS43434_MEMS_Mic -> RevK:ICS43434_MEMS_Mic_Open
Connections:
- net +3V3: now also C20.1
- net +5V: now also C13.2, C17.2, C18.2, C19.2, C21.2, C22.2, C23.2, C24.2, C25.2, C26.2, C27.2, C28.2, C29.2, C30.2, C31.1, D10.2 (+), D11.2 (+), D12.2 (+), D13.2 (+), D14.2 (+), D15.2 (+), D16.2 (+), D17.2 (+), D18.2 (+), D19.2 (+), D20.2 (+), D7.2 (+), D8.2 (+), D9.2 (+)
- net BTN: now also U2.20 (GPIO16), SW1.1 (A); no longer U2.10 (GPIO6)
- net GND: now also C13.1, C17.1, C18.1, C19.1, C20.2, C21.1, C22.1, C23.1, C24.1, C25.1, C26.1, C27.1, C28.1, C29.1, C30.1, C31.2, D10.3 (-), D11.3 (-), D12.3 (-), D13.3 (-), D14.3 (-), D15.3 (-), D16.3 (-), D17.3 (-), D18.3 (-), D19.3 (-), D20.3 (-), D7.3 (-), D8.3 (-), D9.3 (-), SW1.2 (B)
- net LED: now also U2.37 (GPIO41); no longer U2.9 (GPIO5)
- net MICSCK: now also U2.40 (GPIO44); no longer U2.39 (GPIO43)
- net MICSD: now also U2.39 (GPIO43); no longer U2.40 (GPIO44)
- net MICWS: now also U2.38 (GPIO42); no longer U2.44 (GPIO46)
- net SPKBSCK: now also U2.31 (GPIO35); no longer U2.6 (GPIO2)
- net SPKDATA: now also U2.32 (GPIO36); no longer U2.7 (GPIO3)
- net SPKLRC: now also U2.29 (GPIO34); no longer U2.5 (GPIO1)
- net SPKPWR: now also U2.33 (GPIO37); no longer U2.8 (GPIO4)
- net at J2.1 (Pin_1), U6.B3 (OUTN): now also P2.1 (P)
- net at J2.2 (Pin_2), U6.A3 (OUTP): now also P1.1 (P)
- net at D6.1 (O): now also D7.4 (I)
- new net: D17.1 (O), D18.4 (I)
- new net: D16.1 (O), D17.4 (I)
- new net: D8.1 (O), D9.4 (I)
- new net: D7.1 (O), D8.4 (I)
- new net: D19.1 (O), D20.4 (I)
- new net: D18.1 (O), D19.4 (I)
- new net: D10.4 (I), D9.1 (O)
- new net: D10.1 (O), D11.4 (I)
- new net: D15.1 (O), D16.4 (I)
- new net: D11.1 (O), D12.4 (I)
- new net: D13.1 (O), D14.4 (I)
- new net: D12.1 (O), D13.4 (I)
- new net: D14.1 (O), D15.4 (I)
Other:
- title: IronMan Chest -> Intercom
- moved on the sheet: C11, C12, C14, C15, C16, C5, C6, C7, C8, C9, D1, D2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

Commit message: Render
Parts:
- SW1: footprint RevK:SPEH130103 -> Button_Switch_SMD:SW_Push_1TS009xxxx-xxxx-xxxx_6x6x5mm
Changed lines of the file:
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@@
 			)
 		)
-		(property "Footprint" "RevK:SPEH130103"
+		(property "Footprint" "Button_Switch_SMD:SW_Push_1TS009xxxx-xxxx-xxxx_6x6x5mm"
 			(at 139.7 64.77 0)
 			(effects
